File: kastenwagen-pcb/kastenwagen-pcb.kicad_pcb (KiCad board)
At the start: 2 copper layers, 350.5 x 83.5 mm, 111 parts, among them U1 Elite-C

Commit message: On-board MCU to universal daughterboard
Parts:
- added C1: 22pF, Capacitor_SMD:C_0805_2012Metric, B.Cu at (276.7, 45.8)
- added C14: 0.1uF, Capacitor_SMD:C_0805_2012Metric, B.Cu at (286.6, 35.8)
- added C2: 0.1uF, Capacitor_SMD:C_0805_2012Metric, B.Cu at (273.2, 24.1)
- added C24: 0.1uF, Capacitor_SMD:C_0805_2012Metric, B.Cu at (288.3, 18.8)
- added C3: 22pF, Capacitor_SMD:C_0805_2012Metric, B.Cu at (283.4, 45.8)
- added C4: 10uF, Capacitor_SMD:C_0805_2012Metric, B.Cu at (273.2, 22.0)
- added C5: 1uF, Capacitor_SMD:C_0805_2012Metric, B.Cu at (285.2, 17.8)
- added C7: 0.1uF, Capacitor_SMD:C_0805_2012Metric, B.Cu at (274.0, 32.1)
- added F1: 500mA, Fuse:Fuse_1206_3216Metric, B.Cu at (245.5, 25.9)
- added J1: Conn_01x04, random-keyboard-parts:JST-SR-4, B.Cu at (245.6, 18.4)
- added R4: 10k, Keebio-Parts:R_0805, B.Cu at (290.4, 22.6)
- added R5: 22, Keebio-Parts:R_0805, B.Cu at (281.9, 19.2)
- added R6: 22, Keebio-Parts:R_0805, B.Cu at (280.1, 19.2)
- added R7: 10k, Keebio-Parts:R_0805, B.Cu at (276.9, 36.6)
- added SW1: SW_Push, Button_Switch_SMD:SW_Push_1P1T_NO_6x6mm_H9.5mm, B.Cu at (262.6, 63.6)
- added Y1: 16MHz, Crystal:Crystal_SMD_3225-4Pin_3.2x2.5mm, B.Cu at (280.1, 45.8)
- U1: value Elite-C -> ATmega32U4-AU; footprint Keebio-Parts:Elite-C-castellated-29pin-holes -> Package_QFP:TQFP-44_10x10mm_P0.8mm
- moved R3 12.1 mm to (286.6, 39.2)
- moved U1 3.62 mm to (282.5, 28.0)
Connections:
- U1 pad 1: Rotary1A -> Col7
- U1 pad 10: Col7 -> Col6
- U1 pad 11: Row0 -> Col5
- U1 pad 12: Row1 -> Row2
- U1 pad 13: Row7 -> Net-(R4-Pad2)
- U1 pad 14: Col6 -> +5V
- U1 pad 15: Col5 -> GND
- U1 pad 16: Col4 -> Net-(C3-Pad1)
- U1 pad 17: Col3 -> Net-(C1-Pad1)
- U1 pad 18: Col2 -> Rotary0A
- U1 pad 19: Col1 -> Rotary0B
- U1 pad 2: Rotary1B -> +5V
- U1 pad 20: Col0 -> Rotary1B
- U1 pad 21: Net-(U1-Pad21) -> Rotary1A
- U1 pad 22: Net-(U1-Pad22) -> Row3
- U1 pad 24: LED1 -> +5V
- U1 pad 25: Row2 -> LED2
- U1 pad 26: Row3 -> Net-(U1-Pad26)
- U1 pad 27: Row4 -> Col8
- U1 pad 28: Row5 -> Row0
- U1 pad 29: Row6 -> Row1
- U1 pad 3: GND -> Net-(R6-Pad2)
- U1 pad 4: GND -> Net-(R5-Pad1)
- U1 pad 5: Rotary0B -> GND
- U1 pad 6: Rotary0A -> Net-(C5-Pad1)
- U1 pad 7: LED2 -> +5V
- U1 pad 8: LED3 -> LED1
- U1 pad 9: Col8 -> Col4
Routing:
- net GND: track 2173.8 -> 1219.4 mm, vias 180 -> 95
- net +5V: track 0.00 -> 102.5 mm, vias 0 -> 6
- net Net-(R4-Pad2): track 0.00 -> 101.6 mm, vias 0 -> 2
- net Col4: track 228.5 -> 270.6 mm, vias 1 -> 3
- net DP: track 0.00 -> 38.8 mm
- net DN: track 0.00 -> 37.6 mm
- net Col8: track 194.8 -> 231.8 mm, vias 0 -> 3
- net Net-(C1-Pad1): track 0.00 -> 33.8 mm, vias 0 -> 2
- net Net-(C3-Pad1): track 0.00 -> 30.8 mm, vias 0 -> 2
- net Col6: track 79.2 -> 105.7 mm, vias 0 -> 3
- net Col2: track 264.8 -> 290.2 mm, vias 1 -> 3
- net Col5: track 191.4 -> 215.1 mm, vias 0 -> 2
- net Row2: track 281.3 -> 304.9 mm, vias 1 -> 2
- net Row3: track 280.9 -> 303.8 mm, vias 1 -> 2
- net Row5: track 296.0 -> 315.1 mm, vias 1 -> 2
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