File: kastenwagen-pcb/kastenwagen-48/kastenwagen-48-pcb.sch (KiCad schematic (older format))
At the start: 111 parts, among them U1 Elite-C

Commit message: Add PCB and Schema for 48
Parts:
- removed D171, D272, D273, D374, D375, D477: BAV70, Keebio-Parts:SOT-23_Handsoldering, symbol Diode:BAV70
- removed MX170, MX171, MX180, MX273, MX282, MX283, MX375, MX384, MX385, MX477, MX486, MX487: MX-NoLED, MX_Only:MXOnly-1U-NoLED, symbol MX_Alps_Hybrid:MX-NoLED
- removed MX477.200: MX-NoLED, MX_Only:MXOnly-2U-ReversedStabilizers-NoLED, symbol MX_Alps_Hybrid:MX-NoLED
- removed MX487.200: MX-NoLED, MX_Only:MXOnly-2U-NoLED, symbol MX_Alps_Hybrid:MX-NoLED
- RSW100: symbol kastenwagen-pcb-rescue:Rotary_Encoder_Switch-Device -> kastenwagen-48-pcb-rescue:Rotary_Encoder_Switch-Device-kastenwagen-pcb-rescue
- RSW170: renamed from RSW181; symbol kastenwagen-pcb-rescue:Rotary_Encoder_Switch-Device -> kastenwagen-48-pcb-rescue:Rotary_Encoder_Switch-Device-kastenwagen-pcb-rescue
- renumbered MX181 to MX170
Connections:
- net labels removed: Col8
- wire segments 301 -> 238
- no-connect marks 5 -> 6
Other:
- moved on the sheet: D476, MX170, MX476
