File: kastenwagen-pcb/kastenwagen-48/kastenwagen-48-pcb.kicad_pcb (KiCad board)
At the start: 2 copper layers, 292.5 x 83.5 mm, 91 parts, among them U1 Elite-C

Commit message: Further gerber updates
Other:
- board text added: "Build Notes: Diodes, Elite C, & Resistors all surface-mount to this side of the PCB (bottom). LEDs should be surface-mounted to the top side. Install LEDs before adding switches."
- board text added: "Kastenwagen PCB NoPunIn10Did Prototype 2021-06"
- board text removed: "Kastenwagen PCB NoPunIn10Did Prototype 2021-04"
