File: kastenwagen-pcb/kastenwagen-48/kastenwagen-48-plate/kastenwagen-48-bottom.kicad_pcb (KiCad board)
At the start: 2 copper layers, 299.4 x 89.5 mm, 0 parts

Commit message: Updated plate bezels and gerbers
Other:
- board size 299.4 x 89.5 mm -> 303.9 x 94.5 mm
Changed lines of the file:
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@@
   (general
     (thickness 1.6)
-    (drawings 123)
+    (drawings 120)
     (tracks 0)
     (zones 0)
@@
     (uvia_drill 0.1)
   )
+  (gr_arc (start 302.85 88.5) (end 302.85 93.5) (angle -90) (layer Dwgs.User) (width 0.2))
+  (gr_line (start 307.85 15) (end 307.85 88.5) (layer Dwgs.User) (width 0.2))
+  (gr_arc (start 302.85 15) (end 307.85 15) (angle -90) (layer Dwgs.User) (width 0.2))
+  (gr_circle (center 175.75 8) (end 176.9 8) (layer Edge.Cuts) (width 0.15))
+  (gr_line (start 14.5 15) (end 14.5 88.5) (layer Dwgs.User) (width 0.2))
+  (gr_circle (center 175.75 8) (end 176.55 8) (layer Dwgs.User) (width 0.15))
+  (gr_circle (center 14 9.5) (end 14.8 9.5) (layer Dwgs.User) (width 0.15))
+  (gr_arc (start 14 9.5) (end 14 4.5) (angle -90) (layer Edge.Cuts) (width 0.2))
+  (gr_line (start 9 94) (end 9 9.5) (layer Edge.Cuts) (width 0.2))
+  (gr_line (start 19.5 93.5) (end 302.85 93.5) (layer Dwgs.User) (width 0.2))
+  (gr_line (start 14 99) (end 307.85 99) (layer Edge.Cuts) (width 0.2))
+  (gr_circle (center 175.75 95.5) (end 176.9 95.5) (layer Edge.Cuts) (width 0.15))
+  (gr_line (start 19.5 10) (end 302.85 10) (layer Dwgs.User) (width 0.2))
+  (gr_line (start 14 4.5) (end 307.85 4.5) (layer Edge.Cuts) (width 0.2))
+  (gr_circle (center 14 9.5) (end 15.15 9.5) (layer Edge.Cuts) (width 0.15))
+  (gr_line (start 312.85 94) (end 312.85 9.5) (layer Edge.Cuts) (width 0.2))
+  (gr_arc (start 14 94) (end 9 94) (angle -90) (layer Edge.Cuts) (width 0.2))
+  (gr_arc (start 19.5 15) (end 19.5 10) (angle -90) (layer Dwgs.User) (width 0.2))
+  (gr_arc (start 19.5 88.5) (end 14.5 88.5) (angle -90) (layer Dwgs.User) (width 0.2))
+  (gr_circle (center 14 94) (end 15.15 94) (layer Edge.Cuts) (width 0.15))
+  (gr_circle (center 307.85 94) (end 308.65 94) (layer Dwgs.User) (width 0.15))
+  (gr_arc (start 307.85 94) (end 307.85 99) (angle -90) (layer Edge.Cuts) (width 0.2))
+  (gr_circle (center 14 94) (end 14.8 94) (layer Dwgs.User) (width 0.15))
+  (gr_circle (center 307.85 9.5) (end 308.65 9.5) (layer Dwgs.User) (width 0.15))
+  (gr_circle (center 307.85 94) (end 309 94) (layer Edge.Cuts) (width 0.15))
+  (gr_circle (center 307.85 9.5) (end 309 9.5) (layer Edge.Cuts) (width 0.15))
+  (gr_arc (start 307.85 9.5) (end 312.85 9.5) (angle -90) (layer Edge.Cuts) (width 0.2))
+  (gr_circle (center 175.75 95.5) (end 176.55 95.5) (layer Dwgs.User) (width 0.15))
   (gr_line (start 289.14125 87.98627) (end 288.8825 86.92877) (layer B.SilkS) (width 0.2))
   (gr_line (start 289.8725 88.90877) (end 289.14125 87.98627) (layer B.SilkS) (width 0.2))
@@
     (effects (font (size 1.5 1.5) (thickness 0.3)) (justify left))
   )
-  (gr_circle (center 307.85 10) (end 309 10) (layer Edge.Cuts) (width 0.15))
-  (gr_line (start 310.85 91.5) (end 310.85 12) (layer Edge.Cuts) (width 0.2))
-  (gr_circle (center 307.85 93.5) (end 308.65 93.5) (layer Dwgs.User) (width 0.15))
-  (gr_arc (start 305.85 91.5) (end 305.85 96.5) (angle -90) (layer Edge.Cuts) (width 0.2))
-  (gr_arc (start 305.85 12) (end 310.85 12) (angle -90) (layer Edge.Cuts) (width 0.2))
-  (gr_circle (center 307.85 93.5) (end 309 93.5) (layer Edge.Cuts) (width 0.15))
-  (gr_arc (start 302.85 15) (end 307.85 15) (angle -90) (layer Dwgs.User) (width 0.2))
-  (gr_line (start 307.85 15) (end 307.85 88.5) (layer Dwgs.User) (width 0.2))
-  (gr_arc (start 302.85 88.5) (end 302.85 93.5) (angle -90) (layer Dwgs.User) (width 0.2))
-  (gr_circle (center 307.85 10) (end 308.65 10) (layer Dwgs.User) (width 0.15))
-  (gr_circle (center 14.5 93.5) (end 15.3 93.5) (layer Dwgs.User) (width 0.15))
-  (gr_circle (center 14.5 10) (end 15.3 10) (layer Dwgs.User) (width 0.15))
-  (gr_circle (center 175.75 8.5) (end 176.55 8.5) (layer Dwgs.User) (width 0.15))
-  (gr_circle (center 175.75 95) (end 176.55 95) (layer Dwgs.User) (width 0.15))
-  (gr_arc (start 16.5 12) (end 16.5 7) (angle -90) (layer Edge.Cuts) (width 0.2))
-  (gr_line (start 11.5 91.5) (end 11.5 12) (layer Edge.Cuts) (width 0.2))
-  (gr_arc (start 16.5 91.5) (end 11.5 91.5) (angle -90) (layer Edge.Cuts) (width 0.2))
-  (gr_line (start 16.5 7) (end 305.85 7) (layer Edge.Cuts) (width 0.2))
-  (gr_line (start 16.5 96.5) (end 305.85 96.5) (layer Edge.Cuts) (width 0.2))
-  (gr_circle (center 175.75 95) (end 176.9 95) (layer Edge.Cuts) (width 0.15))
-  (gr_circle (center 14.5 93.5) (end 15.65 93.5) (layer Edge.Cuts) (width 0.15))
-  (gr_circle (center 14.5 10) (end 15.65 10) (layer Edge.Cuts) (width 0.15))
-  (gr_circle (center 175.75 8.5) (end 176.9 8.5) (layer Edge.Cuts) (width 0.15))
-  (gr_circle (center 282.6004 18.2364) (end 283.1004 18.2364) (layer Edge.Cuts) (width 0.2))
-  (gr_circle (center 282.6004 27.7364) (end 283.1004 27.7364) (layer Edge.Cuts) (width 0.2))
-  (gr_circle (center 282.6004 37.2364) (end 283.1004 37.2364) (layer Edge.Cuts) (width 0.2))
-  (gr_line (start 14.5 15) (end 14.5 88.5) (layer Dwgs.User) (width 0.2))
-  (gr_arc (start 19.5 15) (end 19.5 10) (angle -90) (layer Dwgs.User) (width 0.2))
-  (gr_line (start 19.5 10) (end 302.85 10) (layer Dwgs.User) (width 0.2))
-  (gr_line (start 19.5 93.5) (end 302.85 93.5) (layer Dwgs.User) (width 0.2))
-  (gr_arc (start 19.5 88.5) (end 14.5 88.5) (angle -90) (layer Dwgs.User) (width 0.2))
+  (zone (net 0) (net_name "") (layer F.Cu) (hatch edge 0.508)
+    (connect_pads (clearance 0.508))
+    (min_thickness 0.254)
+    (fill yes (arc_segments 32) (thermal_gap 0.508) (thermal_bridge_width 0.508) (smoothing fillet))
+    (polygon
+      (pts
+        (xy 375 105) (xy -1.25 105) (xy 0.25 2.5) (xy 375 2.5)
+      )
+    )
+  )
   (zone (net 0) (net_name "") (layer B.Cu) (hatch edge 0.508)
     (connect_pads (clearance 0.508))
@@
     (polygon
       (pts
-        (xy 369.5 98.25) (xy 11 98.25) (xy 11 5.75) (xy 369.5 5.75)
+        (xy 375 105) (xy -1.25 105) (xy 0.25 2.5) (xy 375 2.5)
       )
     )
-  )
-  (zone (net 0) (net_name "") (layer F.Cu) (hatch edge 0.508)
-    (connect_pads (clearance 0.508))
-    (min_thickness 0.254)
-    (fill yes (arc_segments 32) (thermal_gap 0.508) (thermal_bridge_width 0.508) (smoothing fillet))
-    (polygon
-      (pts
-        (xy 369.5 98.25) (xy 11 98.25) (xy 11 5.75) (xy 369.5 5.75)
-      )
-    )
