File: kastenwagen-pcb/kastenwagen-48/kastenwagen-48-plate/kastenwagen-plate.kicad_pcb (KiCad board)
At the start: 2 copper layers, 299.4 x 89.5 mm, 50 parts

Commit message: Updated plate bezels and gerbers
Other:
- board size 299.4 x 89.5 mm -> 303.9 x 94.5 mm
