File: kastenwagen-pcb/kastenwagen-plate/kastenwagen-bottom-plate.kicad_pcb (KiCad board)
At the start: 2 copper layers, 356.5 x 89.5 mm, 0 parts

Commit message: Kastenwagen 1840 plate gerbers
Other:
- board text added: "Kastenwagen 1840: Prototype June 2021 Developed by NoPunIn10Did"
- board text added: "Kastenwagen 1840: Prototype June 2021 Developed by NoPunIn10Did This side toward PCB."
Changed lines of the file:
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@@
   (general
     (thickness 1.6)
-    (drawings 22)
+    (drawings 114)
     (tracks 0)
     (zones 0)
@@
     (visible_elements 7FFFFFFF)
     (pcbplotparams
-      (layerselection 0x010fc_ffffffff)
-      (usegerberextensions false)
-      (usegerberattributes true)
+      (layerselection 0x010f0_ffffffff)
+      (usegerberextensions true)
+      (usegerberattributes false)
       (usegerberadvancedattributes true)
-      (creategerberjobfile true)
+      (creategerberjobfile false)
       (excludeedgelayer true)
-      (linewidth 0.100000)
+      (linewidth 0.020000)
       (plotframeref false)
       (viasonmask false)
@@
       (outputformat 1)
       (mirror false)
-      (drillshape 1)
+      (drillshape 0)
       (scaleselection 1)
-      (outputdirectory ""))
+      (outputdirectory "kastenwagen-1840-bottom-gerbers/"))
   )
   (net 0 "")
@@
     (uvia_drill 0.1)
   )
+  (gr_text "Kastenwagen 1840: Prototype June 2021\nDeveloped by NoPunIn10Did\nThis side toward PCB." (at 315.11875 83.34375) (layer F.SilkS)
+    (effects (font (size 1.5 1.5) (thickness 0.3)) (justify left))
+  )
+  (gr_text "Kastenwagen 1840: Prototype June 2021\nDeveloped by NoPunIn10Did" (at 65.0875 84.93125) (layer B.SilkS)
+    (effects (font (size 1.5 1.5) (thickness 0.3)) (justify left mirror))
+  )
+  (gr_line (start 350.30125 70.76002) (end 351.775 71.00752) (layer B.SilkS) (width 0.2))
+  (gr_line (start 333.74125 75.08002) (end 333.74125 87.56002) (layer B.SilkS) (width 0.2))
+  (gr_line (start 331.58875 68.56627) (end 332.24125 67.43002) (layer B.SilkS) (width 0.2))
+  (gr_line (start 336.62125 75.08002) (end 333.74125 75.08002) (layer B.SilkS) (width 0.2))
+  (gr_line (start 336.62125 87.56002) (end 336.62125 75.08002) (layer B.SilkS) (width 0.2))
+  (gr_line (start 338.815 90.19252) (end 339.95125 89.54002) (layer B.SilkS) (width 0.2))
+  (gr_line (start 335.8675 90.19252) (end 337.34125 90.44002) (layer B.SilkS) (width 0.2))
+  (gr_line (start 338.06125 87.56002) (end 336.62125 87.56002) (layer B.SilkS) (width 0.2))
+  (gr_line (start 334 88.61752) (end 334.73125 89.54002) (layer B.SilkS) (width 0.2))
+  (gr_line (start 331.58875 71.51377) (end 331.34125 70.04002) (layer B.SilkS) (width 0.2))
+  (gr_line (start 332.24125 72.65002) (end 331.58875 71.51377) (layer B.SilkS) (width 0.2))
+  (gr_line (start 340.94125 75.08002) (end 338.06125 75.08002) (layer B.SilkS) (width 0.2))
+  (gr_line (start 334.73125 89.54002) (end 335.8675 90.19252) (layer B.SilkS) (width 0.2))
+  (gr_line (start 334.22125 66.44002) (end 353.90125 66.44002) (layer B.SilkS) (width 0.2))
+  (gr_line (start 342.38125 73.64002) (end 334.22125 73.64002) (layer B.SilkS) (width 0.2))
+  (gr_line (start 339.95125 89.54002) (end 340.6825 88.61752) (layer B.SilkS) (width 0.2))
+  (gr_line (start 337.34125 90.44002) (end 338.815 90.19252) (layer B.SilkS) (width 0.2))
+  (gr_line (start 333.74125 87.56002) (end 334 88.61752) (layer B.SilkS) (width 0.2))
+  (gr_line (start 334.22125 73.64002) (end 333.16375 73.38127) (layer B.SilkS) (width 0.2))
+  (gr_line (start 353.90125 87.56002) (end 353.6425 88.61752) (layer B.SilkS) (width 0.2))
+  (gr_line (start 353.90125 73.64002) (end 353.90125 87.56002) (layer B.SilkS) (width 0.2))
+  (gr_line (start 352.91125 71.66002) (end 353.6425 72.58252) (layer B.SilkS) (width 0.2))
+  (gr_line (start 333.16375 73.38127) (end 332.24125 72.65002) (layer B.SilkS) (width 0.2))
+  (gr_line (start 353.6425 72.58252) (end 353.90125 73.64002) (layer B.SilkS) (width 0.2))
+  (gr_line (start 351.775 71.00752) (end 352.91125 71.66002) (layer B.SilkS) (width 0.2))
+  (gr_line (start 340.6825 88.61752) (end 340.94125 87.56002) (layer B.SilkS) (width 0.2))
+  (gr_line (start 333.16375 66.69877) (end 334.22125 66.44002) (layer B.SilkS) (width 0.2))
+  (gr_line (start 338.06125 75.08002) (end 338.06125 87.56002) (layer B.SilkS) (width 0.2))
+  (gr_line (start 340.94125 87.56002) (end 340.94125 75.08002) (layer B.SilkS) (width 0.2))
+  (gr_line (start 345.26125 87.56002) (end 342.38125 87.56002) (layer B.SilkS) (width 0.2))
+  (gr_line (start 332.24125 67.43002) (end 333.16375 66.69877) (layer B.SilkS) (width 0.2))
+  (gr_line (start 342.38125 87.56002) (end 342.38125 73.64002) (layer B.SilkS) (width 0.2))
+  (gr_line (start 331.34125 70.04002) (end 331.58875 68.56627) (layer B.SilkS) (width 0.2))
+  (gr_line (start 345.26125 73.64002) (end 345.26125 87.56002) (layer B.SilkS) (width 0.2))
+  (gr_line (start 350.30125 90.44002) (end 348.8275 90.19252) (layer B.SilkS) (width 0.2))
+  (gr_line (start 362.2825 68.26252) (end 362.54125 69.32002) (layer B.SilkS) (width 0.2))
+  (gr_line (start 351.02125 87.56002) (end 351.02125 73.64002) (layer B.SilkS) (width 0.2))
+  (gr_line (start 351.02125 73.64002) (end 349.58125 73.64002) (layer B.SilkS) (width 0.2))
+  (gr_line (start 361.55125 67.34002) (end 362.2825 68.26252) (layer B.SilkS) (width 0.2))
+  (gr_line (start 360.415 66.68752) (end 361.55125 67.34002) (layer B.SilkS) (width 0.2))
+  (gr_line (start 358.94125 66.44002) (end 360.415 66.68752) (layer B.SilkS) (width 0.2))
+  (gr_line (start 348.8275 71.00752) (end 350.30125 70.76002) (layer B.SilkS) (width 0.2))
+  (gr_line (start 347.69125 89.54002) (end 346.96 88.61752) (layer B.SilkS) (width 0.2))
+  (gr_line (start 346.70125 73.64002) (end 346.96 72.58252) (layer B.SilkS) (width 0.2))
+  (gr_line (start 346.96 88.61752) (end 346.70125 87.56002) (layer B.SilkS) (width 0.2))
+  (gr_line (start 351.775 90.19252) (end 350.30125 90.44002) (layer B.SilkS) (width 0.2))
+  (gr_line (start 353.6425 88.61752) (end 352.91125 89.54002) (layer B.SilkS) (width 0.2))
+  (gr_line (start 352.91125 89.54002) (end 351.775 90.19252) (layer B.SilkS) (width 0.2))
+  (gr_line (start 346.96 72.58252) (end 347.69125 71.66002) (layer B.SilkS) (width 0.2))
+  (gr_line (start 346.70125 87.56002) (end 346.70125 73.64002) (layer B.SilkS) (width 0.2))
+  (gr_line (start 348.8275 90.19252) (end 347.69125 89.54002) (layer B.SilkS) (width 0.2))
+  (gr_line (start 347.69125 71.66002) (end 348.8275 71.00752) (layer B.SilkS) (width 0.2))
+  (gr_line (start 350.30125 70.76002) (end 350.30125 70.76002) (layer B.SilkS) (width 0.2))
+  (gr_line (start 349.58125 87.56002) (end 351.02125 87.56002) (layer B.SilkS) (width 0.2))
+  (gr_line (start 349.58125 73.64002) (end 349.58125 87.56002) (layer B.SilkS) (width 0.2))
+  (gr_line (start 328.70125 72.20002) (end 330.175 72.44752) (layer B.SilkS) (width 0.2))
+  (gr_line (start 327.2275 72.44752) (end 328.70125 72.20002) (layer B.SilkS) (width 0.2))
+  (gr_line (start 325.10125 90.44002) (end 325.10125 75.08002) (layer B.SilkS) (width 0.2))
+  (gr_line (start 330.175 72.44752) (end 331.31125 73.10002) (layer B.SilkS) (width 0.2))
+  (gr_line (start 332.0425 74.02252) (end 332.30125 75.08002) (layer B.SilkS) (width 0.2))
+  (gr_line (start 327.98125 90.44002) (end 325.10125 90.44002) (layer B.SilkS) (width 0.2))
+  (gr_line (start 332.30125 87.56002) (end 329.42125 87.56002) (layer B.SilkS) (width 0.2))
+  (gr_line (start 329.42125 75.08002) (end 327.98125 75.08002) (layer B.SilkS) (width 0.2))
+  (gr_line (start 326.09125 73.10002) (end 327.2275 72.44752) (layer B.SilkS) (width 0.2))
+  (gr_line (start 329.42125 87.56002) (end 329.42125 75.08002) (layer B.SilkS) (width 0.2))
+  (gr_line (start 332.30125 75.08002) (end 332.30125 87.56002) (layer B.SilkS) (width 0.2))
+  (gr_line (start 331.31125 73.10002) (end 332.0425 74.02252) (layer B.SilkS) (width 0.2))
+  (gr_line (start 327.98125 75.08002) (end 327.98125 90.44002) (layer B.SilkS) (width 0.2))
+  (gr_line (start 345.01375 72.58252) (end 345.26125 73.64002) (layer B.SilkS) (width 0.2))
+  (gr_line (start 344.36125 71.66002) (end 345.01375 72.58252) (layer B.SilkS) (width 0.2))
+  (gr_line (start 334.22125 70.76002) (end 342.38125 70.76002) (layer B.SilkS) (width 0.2))
+  (gr_line (start 353.90125 69.32002) (end 334.22125 69.32002) (layer B.SilkS) (width 0.2))
+  (gr_line (start 343.43875 71.00752) (end 344.36125 71.66002) (layer B.SilkS) (width 0.2))
+  (gr_line (start 342.38125 70.76002) (end 343.43875 71.00752) (layer B.SilkS) (width 0.2))
+  (gr_line (start 334.22125 69.32002) (end 334.22125 70.76002) (layer B.SilkS) (width 0.2))
+  (gr_line (start 353.90125 66.44002) (end 353.90125 69.32002) (layer B.SilkS) (width 0.2))
+  (gr_line (start 359.66125 90.44002) (end 359.66125 69.31992) (layer B.SilkS) (width 0.2))
+  (gr_line (start 355.34125 69.32) (end 355.6 68.2625) (layer B.SilkS) (width 0.2))
+  (gr_line (start 355.34131 87.56) (end 355.34125 69.32) (layer B.SilkS) (width 0.2))
+  (gr_line (start 358.22125 69.32) (end 358.22125 87.56) (layer B.SilkS) (width 0.2))
+  (gr_line (start 358.22125 87.56) (end 355.34131 87.56) (layer B.SilkS) (width 0.2))
+  (gr_line (start 325.359999 74.02252) (end 326.09125 73.10002) (layer B.SilkS) (width 0.2))
+  (gr_line (start 359.66125 69.31992) (end 358.22125 69.32) (layer B.SilkS) (width 0.2))
+  (gr_line (start 358.94125 66.44) (end 358.94125 66.44002) (layer B.SilkS) (width 0.2))
+  (gr_line (start 357.4675 66.6875) (end 358.94125 66.44) (layer B.SilkS) (width 0.2))
+  (gr_line (start 362.54125 90.44002) (end 359.66125 90.44002) (layer B.SilkS) (width 0.2))
+  (gr_line (start 362.54125 69.32002) (end 362.54125 90.44002) (layer B.SilkS) (width 0.2))
+  (gr_line (start 325.10125 75.08002) (end 325.359999 74.02252) (layer B.SilkS) (width 0.2))
+  (gr_line (start 356.33125 67.34) (end 357.4675 66.6875) (layer B.SilkS) (width 0.2))
+  (gr_line (start 355.6 68.2625) (end 356.33125 67.34) (layer B.SilkS) (width 0.2))
   (gr_arc (start 16.5 12) (end 16.5 7) (angle -90) (layer Edge.Cuts) (width 0.2))
   (gr_line (start 11.5 91.5) (end 11.5 12) (layer Edge.Cuts) (width 0.2))

Commit message: Further gerber updates
Other:
- board text added: "Kastenwagen 1840: Prototype 2021-06 Developed by NoPunIn10Did"
- board text added: "Kastenwagen 1840: Prototype 2021-06 Developed by NoPunIn10Did This side toward PCB."
- board text removed: "Kastenwagen 1840: Prototype June 2021 Developed by NoPunIn10Did"
- board text removed: "Kastenwagen 1840: Prototype June 2021 Developed by NoPunIn10Did This side toward PCB."
Changed lines of the file:
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@@
     (uvia_drill 0.1)
   )
-  (gr_text "Kastenwagen 1840: Prototype June 2021\nDeveloped by NoPunIn10Did\nThis side toward PCB." (at 315.11875 83.34375) (layer F.SilkS)
+  (gr_text "Kastenwagen 1840: Prototype 2021-06\nDeveloped by NoPunIn10Did\nThis side toward PCB." (at 315.11875 83.34375) (layer F.SilkS)
     (effects (font (size 1.5 1.5) (thickness 0.3)) (justify left))
   )
-  (gr_text "Kastenwagen 1840: Prototype June 2021\nDeveloped by NoPunIn10Did" (at 65.0875 84.93125) (layer B.SilkS)
+  (gr_text "Kastenwagen 1840: Prototype 2021-06\nDeveloped by NoPunIn10Did" (at 65.0875 84.93125) (layer B.SilkS)
     (effects (font (size 1.5 1.5) (thickness 0.3)) (justify left mirror))
   )

Commit message: Updated plate bezels and gerbers
Other:
- board size 356.5 x 89.5 mm -> 361.5 x 94.5 mm
Changed lines of the file:
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@@
   (general
     (thickness 1.6)
-    (drawings 114)
+    (drawings 120)
     (tracks 0)
     (zones 0)
@@
     (uvia_drill 0.1)
   )
+  (gr_circle (center 175.75 95.5) (end 176.55 95.5) (layer Dwgs.User) (width 0.15))
+  (gr_circle (center 365.5 94) (end 366.3 94) (layer Dwgs.User) (width 0.15))
+  (gr_circle (center 365.5 9.5) (end 366.3 9.5) (layer Dwgs.User) (width 0.15))
+  (gr_circle (center 14 94) (end 14.8 94) (layer Dwgs.User) (width 0.15))
+  (gr_circle (center 175.75 8) (end 176.55 8) (layer Dwgs.User) (width 0.15))
+  (gr_circle (center 14 9.5) (end 14.8 9.5) (layer Dwgs.User) (width 0.15))
+  (gr_arc (start 14 94) (end 9 94) (angle -90) (layer Edge.Cuts) (width 0.2))
+  (gr_arc (start 14 9.5) (end 14 4.5) (angle -90) (layer Edge.Cuts) (width 0.2))
+  (gr_line (start 9 94) (end 9 9.5) (layer Edge.Cuts) (width 0.2))
+  (gr_circle (center 365.5 94) (end 366.65 94) (layer Edge.Cuts) (width 0.15))
+  (gr_arc (start 365.5 94) (end 365.5 99) (angle -90) (layer Edge.Cuts) (width 0.2))
+  (gr_arc (start 360 88.5) (end 360 93.5) (angle -90) (layer Dwgs.User) (width 0.2))
+  (gr_arc (start 19.5 88.5) (end 14.5 88.5) (angle -90) (layer Dwgs.User) (width 0.2))
+  (gr_line (start 19.5 93.5) (end 360 93.5) (layer Dwgs.User) (width 0.2))
+  (gr_circle (center 175.75 8) (end 176.9 8) (layer Edge.Cuts) (width 0.15))
+  (gr_line (start 19.5 10) (end 360 10) (layer Dwgs.User) (width 0.2))
+  (gr_line (start 14 4.5) (end 365.5 4.5) (layer Edge.Cuts) (width 0.2))
+  (gr_circle (center 365.5 9.5) (end 366.65 9.5) (layer Edge.Cuts) (width 0.15))
+  (gr_arc (start 19.5 15) (end 19.5 10) (angle -90) (layer Dwgs.User) (width 0.2))
+  (gr_circle (center 175.75 95.5) (end 176.9 95.5) (layer Edge.Cuts) (width 0.15))
+  (gr_line (start 14.5 15) (end 14.5 88.5) (layer Dwgs.User) (width 0.2))
+  (gr_arc (start 360 15) (end 365 15) (angle -90) (layer Dwgs.User) (width 0.2))
+  (gr_line (start 365 15) (end 365 88.5) (layer Dwgs.User) (width 0.2))
+  (gr_circle (center 14 9.5) (end 15.15 9.5) (layer Edge.Cuts) (width 0.15))
+  (gr_circle (center 14 94) (end 15.15 94) (layer Edge.Cuts) (width 0.15))
+  (gr_line (start 370.5 94) (end 370.5 9.5) (layer Edge.Cuts) (width 0.2))
+  (gr_arc (start 365.5 9.5) (end 370.5 9.5) (angle -90) (layer Edge.Cuts) (width 0.2))
+  (gr_line (start 14 99) (end 365.5 99) (layer Edge.Cuts) (width 0.2))
   (gr_text "Kastenwagen 1840: Prototype 2021-06\nDeveloped by NoPunIn10Did\nThis side toward PCB." (at 315.11875 83.34375) (layer F.SilkS)
     (effects (font (size 1.5 1.5) (thickness 0.3)) (justify left))
@@
   (gr_line (start 356.33125 67.34) (end 357.4675 66.6875) (layer B.SilkS) (width 0.2))
   (gr_line (start 355.6 68.2625) (end 356.33125 67.34) (layer B.SilkS) (width 0.2))
-  (gr_arc (start 16.5 12) (end 16.5 7) (angle -90) (layer Edge.Cuts) (width 0.2))
-  (gr_line (start 11.5 91.5) (end 11.5 12) (layer Edge.Cuts) (width 0.2))
-  (gr_arc (start 16.5 91.5) (end 11.5 91.5) (angle -90) (layer Edge.Cuts) (width 0.2))
-  (gr_line (start 16.5 7) (end 363 7) (layer Edge.Cuts) (width 0.2))
-  (gr_arc (start 363 12) (end 368 12) (angle -90) (layer Edge.Cuts) (width 0.2))
-  (gr_line (start 16.5 96.5) (end 363 96.5) (layer Edge.Cuts) (width 0.2))
-  (gr_line (start 368 91.5) (end 368 12) (layer Edge.Cuts) (width 0.2))
-  (gr_arc (start 363 91.5) (end 363 96.5) (angle -90) (layer Edge.Cuts) (width 0.2))
-  (gr_circle (center 175.75 95) (end 176.9 95) (layer Edge.Cuts) (width 0.15))
-  (gr_circle (center 14.5 93.5) (end 15.65 93.5) (layer Edge.Cuts) (width 0.15))
-  (gr_circle (center 14.5 10) (end 15.65 10) (layer Edge.Cuts) (width 0.15))
-  (gr_circle (center 365 93.5) (end 366.15 93.5) (layer Edge.Cuts) (width 0.15))
-  (gr_circle (center 365 10) (end 366.15 10) (layer Edge.Cuts) (width 0.15))
-  (gr_circle (center 175.75 8.5) (end 176.9 8.5) (layer Edge.Cuts) (width 0.15))
-  (gr_line (start 365 15) (end 365 88.5) (layer Dwgs.User) (width 0.2))
-  (gr_arc (start 360 15) (end 365 15) (angle -90) (layer Dwgs.User) (width 0.2))
-  (gr_line (start 14.5 15) (end 14.5 88.5) (layer Dwgs.User) (width 0.2))
-  (gr_arc (start 19.5 15) (end 19.5 10) (angle -90) (layer Dwgs.User) (width 0.2))
-  (gr_line (start 19.5 10) (end 360 10) (layer Dwgs.User) (width 0.2))
-  (gr_line (start 19.5 93.5) (end 360 93.5) (layer Dwgs.User) (width 0.2))
-  (gr_arc (start 19.5 88.5) (end 14.5 88.5) (angle -90) (layer Dwgs.User) (width 0.2))
-  (gr_arc (start 360 88.5) (end 360 93.5) (angle -90) (layer Dwgs.User) (width 0.2))
+  (zone (net 0) (net_name "") (layer F.Cu) (hatch edge 0.508)
+    (connect_pads (clearance 0.508))
+    (min_thickness 0.254)
+    (fill yes (arc_segments 32) (thermal_gap 0.508) (thermal_bridge_width 0.508) (smoothing fillet))
+    (polygon
+      (pts
+        (xy 375 105) (xy -1.25 105) (xy 0.25 2.5) (xy 375 2.5)
+      )
+    )
+  )
   (zone (net 0) (net_name "") (layer B.Cu) (hatch edge 0.508)
     (connect_pads (clearance 0.508))
@@
     (polygon
       (pts
-        (xy 369.5 98.25) (xy 11 98.25) (xy 11 5.75) (xy 369.5 5.75)
+        (xy 375 105) (xy -1.25 105) (xy 0.25 2.5) (xy 375 2.5)
       )
     )
-  )
-  (zone (net 0) (net_name "") (layer F.Cu) (hatch edge 0.508)
-    (connect_pads (clearance 0.508))
-    (min_thickness 0.254)
-    (fill yes (arc_segments 32) (thermal_gap 0.508) (thermal_bridge_width 0.508) (smoothing fillet))
-    (polygon
-      (pts
-        (xy 369.5 98.25) (xy 11 98.25) (xy 11 5.75) (xy 369.5 5.75)
-      )
-    )
