File: kastenwagen-pcb/kastenwagen-plate/kastenwagen-plate.kicad_pcb (KiCad board)
At the start: 2 copper layers, 128.3 x 15 mm, 60 parts

Commit message: Reverse the stabilizers
Parts:
- removed the REF** at (130.2, 82.5)
- added REF**: MX_7.00u Reverse 1.00u 2.75u 2.25u 1.00u, MX_plate_cutouts:MX_7.00u_Reverse_1.00u_2.75u_2.25u_1.00u, F.Cu at (130.2, 82.5)
- turned REF** to 270 degrees
- turned REF** to 180 degrees
Other:
- outline, holes or cut-outs redrawn

Commit message: Plate edits and LED positioning
Routing:
- added copper zone on B.Cu, net (none)
- added copper zone on F.Cu, net (none)
Other:
- board size 128.3 x 15 mm -> 356.5 x 89.5 mm

Commit message: Kastenwagen 1840 plate gerbers
Other:
- board text added: "Kastenwagen 1840: Prototype June 2021 Developed by NoPunIn10Did"

Commit message: Further gerber updates
Other:
- board text added: "Kastenwagen 1840: Prototype 2021-06 Developed by NoPunIn10Did"
- board text removed: "Kastenwagen 1840: Prototype June 2021 Developed by NoPunIn10Did"

Commit message: Updated plate bezels and gerbers
Other:
- board size 356.5 x 89.5 mm -> 361.5 x 94.5 mm
Changed lines of the file:
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@@
     (effects (font (size 1 1) (thickness 0.15)) (justify left mirror))
   )
-  (gr_circle (center 14.5 93.5) (end 15.3 93.5) (layer Dwgs.User) (width 0.15))
-  (gr_circle (center 14.5 10) (end 15.3 10) (layer Dwgs.User) (width 0.15))
-  (gr_circle (center 175.75 8.5) (end 176.55 8.5) (layer Dwgs.User) (width 0.15))
-  (gr_circle (center 365 10) (end 365.8 10) (layer Dwgs.User) (width 0.15))
-  (gr_circle (center 365 93.5) (end 365.8 93.5) (layer Dwgs.User) (width 0.15))
-  (gr_circle (center 175.75 95) (end 176.55 95) (layer Dwgs.User) (width 0.15))
-  (gr_arc (start 16.5 12) (end 16.5 7) (angle -90) (layer Edge.Cuts) (width 0.2))
-  (gr_line (start 11.5 91.5) (end 11.5 12) (layer Edge.Cuts) (width 0.2))
-  (gr_arc (start 16.5 91.5) (end 11.5 91.5) (angle -90) (layer Edge.Cuts) (width 0.2))
-  (gr_line (start 16.5 7) (end 363 7) (layer Edge.Cuts) (width 0.2))
-  (gr_arc (start 363 12) (end 368 12) (angle -90) (layer Edge.Cuts) (width 0.2))
-  (gr_line (start 16.5 96.5) (end 363 96.5) (layer Edge.Cuts) (width 0.2))
-  (gr_line (start 368 91.5) (end 368 12) (layer Edge.Cuts) (width 0.2))
-  (gr_arc (start 363 91.5) (end 363 96.5) (angle -90) (layer Edge.Cuts) (width 0.2))
-  (gr_circle (center 175.75 95) (end 176.9 95) (layer Edge.Cuts) (width 0.15))
-  (gr_circle (center 14.5 93.5) (end 15.65 93.5) (layer Edge.Cuts) (width 0.15))
-  (gr_circle (center 14.5 10) (end 15.65 10) (layer Edge.Cuts) (width 0.15))
-  (gr_circle (center 365 93.5) (end 366.15 93.5) (layer Edge.Cuts) (width 0.15))
-  (gr_circle (center 365 10) (end 366.15 10) (layer Edge.Cuts) (width 0.15))
-  (gr_circle (center 175.75 8.5) (end 176.9 8.5) (layer Edge.Cuts) (width 0.15))
+  (gr_circle (center 14 94) (end 14.8 94) (layer Dwgs.User) (width 0.15))
+  (gr_circle (center 14 9.5) (end 14.8 9.5) (layer Dwgs.User) (width 0.15))
+  (gr_circle (center 175.75 8) (end 176.55 8) (layer Dwgs.User) (width 0.15))
+  (gr_circle (center 365.5 9.5) (end 366.3 9.5) (layer Dwgs.User) (width 0.15))
+  (gr_circle (center 365.5 94) (end 366.3 94) (layer Dwgs.User) (width 0.15))
+  (gr_circle (center 175.75 95.5) (end 176.55 95.5) (layer Dwgs.User) (width 0.15))
+  (gr_arc (start 14 9.5) (end 14 4.5) (angle -90) (layer Edge.Cuts) (width 0.2))
+  (gr_line (start 9 94) (end 9 9.5) (layer Edge.Cuts) (width 0.2))
+  (gr_arc (start 14 94) (end 9 94) (angle -90) (layer Edge.Cuts) (width 0.2))
+  (gr_line (start 14 4.5) (end 365.5 4.5) (layer Edge.Cuts) (width 0.2))
+  (gr_arc (start 365.5 9.5) (end 370.5 9.5) (angle -90) (layer Edge.Cuts) (width 0.2))
+  (gr_line (start 14 99) (end 365.5 99) (layer Edge.Cuts) (width 0.2))
+  (gr_line (start 370.5 94) (end 370.5 9.5) (layer Edge.Cuts) (width 0.2))
+  (gr_arc (start 365.5 94) (end 365.5 99) (angle -90) (layer Edge.Cuts) (width 0.2))
+  (gr_circle (center 175.75 95.5) (end 176.9 95.5) (layer Edge.Cuts) (width 0.15))
+  (gr_circle (center 14 94) (end 15.15 94) (layer Edge.Cuts) (width 0.15))
+  (gr_circle (center 14 9.5) (end 15.15 9.5) (layer Edge.Cuts) (width 0.15))
+  (gr_circle (center 365.5 94) (end 366.65 94) (layer Edge.Cuts) (width 0.15))
+  (gr_circle (center 365.5 9.5) (end 366.65 9.5) (layer Edge.Cuts) (width 0.15))
+  (gr_circle (center 175.75 8) (end 176.9 8) (layer Edge.Cuts) (width 0.15))
   (gr_circle (center 282.6004 18.2364) (end 283.1004 18.2364) (layer Edge.Cuts) (width 0.2))
   (gr_circle (center 282.6004 27.7364) (end 283.1004 27.7364) (layer Edge.Cuts) (width 0.2))
@@
     (polygon
       (pts
-        (xy 369.5 98.25) (xy 11 98.25) (xy 11 5.75) (xy 369.5 5.75)
+        (xy 375 105) (xy -1.25 105) (xy 0.25 2.5) (xy 375 2.5)
       )
     )
@@
     (polygon
       (pts
-        (xy 369.5 98.25) (xy 11 98.25) (xy 11 5.75) (xy 369.5 5.75)
+        (xy 375 105) (xy -1.25 105) (xy 0.25 2.5) (xy 375 2.5)
       )
     )
