File: kastenwagen-1840-pcb/kastenwagen-1840-pcb.kicad_pcb (KiCad board)
At the start: 2 copper layers, 350.5 x 83.5 mm, 111 parts, among them U1 Elite-C

Commit message: redoing traces
Parts:
- moved D476 24.2 mm to (304.3, 81.3)
- moved D437 18.7 mm to (177.2, 78.9)
- moved D262 17.6 mm to (251.5, 40.8)
- moved R1 14.1 mm to (292.4, 18.0), turned to 90 degrees
- moved D160 14.0 mm to (244.5, 21.8)
- moved D304 13.5 mm to (47.2, 59.8)
- moved R3 12.9 mm to (296.8, 20.0), turned to 90 degrees
- moved D477 12.1 mm to (344.4, 77.1)
- moved D305 11.6 mm to (68.2, 59.8)
- moved D223 11.6 mm to (134.9, 40.8)
- moved D325 11.6 mm to (144.4, 59.8)
- moved D273 11.6 mm to (325.4, 40.8)
- moved D375 11.6 mm to (325.4, 59.8)
- moved D243 11.5 mm to (211.1, 40.8)
- moved D203 11.5 mm to (58.8, 40.8)
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Connections:
- D160 pad 1: Net-(D160-Pad1) -> unconnected-(D160-Pad1)
- D262 pad 1: Net-(D262-Pad1) -> unconnected-(D262-Pad1)
- D364 pad 2: Net-(D364-Pad2) -> unconnected-(D364-Pad2)
- MX262 pad 2: Net-(D262-Pad1) -> Net-(D262-Pad2)
- U1 pad 21: Net-(U1-Pad21) -> unconnected-(U1-Pad21)
- U1 pad 22: Net-(U1-Pad22) -> unconnected-(U1-Pad22)
Routing:
- net GND: track 2173.8 -> 392.3 mm, vias 180 -> 13
- net Col0: track 415.8 -> 196.9 mm, vias 0 -> 12
- net Col4: track 228.5 -> 23.3 mm
- net Col8: track 194.8 -> 13.6 mm
- net Col5: track 191.4 -> 21.4 mm, vias 0 -> 1
- net Col1: track 370.4 -> 214.6 mm, vias 1 -> 7
- net Col7: track 164.0 -> 17.2 mm, vias 0 -> 1
- net Col2: track 264.8 -> 161.2 mm, vias 1 -> 9
- net Col3: track 240.5 -> 145.6 mm, vias 1 -> 4
- net Col6: track 79.2 -> 19.5 mm, vias 0 -> 1
- net Row0: track 285.3 -> 340.0 mm, vias 2 -> 16
- net Row1: track 282.4 -> 336.4 mm, vias 2 -> 13
- net Row6: track 352.5 -> 313.9 mm, vias 1 -> 6
- net Rotary0A: track 269.9 -> 304.4 mm, vias 0 -> 4
- net Rotary0B: track 267.1 -> 300.5 mm, vias 0 -> 4
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Other:
- net class Default removed
- net class Power removed
- board text added: "Kastenwagen PCB NoPunIn10Did Prototype 2022-10"
- board text removed: "Kastenwagen PCB NoPunIn10Did Prototype 2021-06"

Commit message: More tracing updates
Routing:
- net GND: track 392.3 -> 1967.7 mm, vias 13 -> 154
- net Col0: track 196.9 -> 431.2 mm, vias 12 -> 14
- net Col4: track 23.3 -> 251.7 mm, vias 1 -> 14
- net Col8: track 13.6 -> 200.4 mm, vias 0 -> 5
- net Col5: track 21.4 -> 201.5 mm, vias 1 -> 7
- net Col7: track 17.2 -> 179.1 mm, vias 1 -> 9
- net Col1: track 214.6 -> 374.2 mm, vias 7 -> 9
- net Col2: track 161.2 -> 288.9 mm, vias 9 -> 11
- net Col3: track 145.6 -> 231.2 mm
- net Col6: track 19.5 -> 97.7 mm, vias 1 -> 5
- net Row6: track 313.9 -> 338.5 mm, vias 6 -> 9
- net Row5: track 306.8 -> 331.4 mm, vias 8 -> 11
- net Row7: track 337.0 -> 361.2 mm, vias 8 -> 10
- net Rotary0B: track 300.5 -> 277.5 mm
- net Rotary0A: track 304.4 -> 283.5 mm
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