File: kastenwagen-1840-chunky/kastenwagen-1840-chunky.kicad_pcb (KiCad board)
At the start: 2 copper layers, 350.5 x 83.5 mm, 109 parts, among them U1 Elite-C

Commit message: Fix the ISO footprint used and retrace where needed
Parts:
- MX262: footprint mx-custom:MXOnly-ISO-ROTATED-NoLED -> mx-custom:MXOnly-ISO-ROTATED-NoLED-NoStabs
- moved D1 2.40 mm to (280.2, 18.2)
- moved D2 2.40 mm to (280.2, 27.7)
- moved D3 2.40 mm to (280.2, 37.2)
Routing:
- net Col3: track 117.5 -> 238.2 mm, vias 4 -> 8
- net Col1: track 339.9 -> 374.3 mm
- net Col2: track 259.3 -> 289.3 mm, vias 11 -> 13
- net Col0: track 406.8 -> 431.2 mm
- net Row0: track 313.6 -> 333.5 mm, vias 14 -> 16
- net Col4: track 234.5 -> 251.7 mm, vias 14 -> 16
- net Net-(MX262-ROW): track 0.00 -> 10.5 mm, vias 0 -> 1
- net GND: track 1967.7 -> 1962.6 mm, vias 154 -> 155
- net Col6: track 78.7 -> 81.3 mm, vias 5 -> 4
- net LED3: track 11.1 -> 13.5 mm
- net LED2: track 6.76 -> 9.16 mm
- net LED1: track 14.2 -> 11.9 mm
- net LED1R: track 21.5 -> 23.1 mm
- net LED3R: track 46.5 -> 45.2 mm
