File: kastenwagen-1840-chunky/kastenwagen-1840-chunky.kicad_sch (KiCad schematic)
At the start: 109 parts, among them U1 Elite-C

Commit message: Fix the ISO footprint used and retrace where needed
Parts:
- MX262: footprint mx-custom:MXOnly-ISO-ROTATED-NoLED -> mx-custom:MXOnly-ISO-ROTATED-NoLED-NoStabs
Changed lines of the file:
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@@
       (effects (font (size 0.508 0.508)))
     )
-    (property "Footprint" "mx-custom:MXOnly-ISO-ROTATED-NoLED" (at 196.215 73.025 0)
+    (property "Footprint" "mx-custom:MXOnly-ISO-ROTATED-NoLED-NoStabs" (at 196.215 73.025 0)
       (effects (font (size 1.524 1.524)) hide)
     )
